File: rev_a/bus_usb_power.sch (KiCad schematic (older format))
At the start: 18 parts, among them J1 TERMINATE_JUMPER, Q1 FQP47P06, Q2 FQP47P06, SW1 F-426-0020

Commit message: Changed internal references from bus_power to bus_usb_power.
Parts:
- G1: footprint (none) -> Bus_Usb_Power:OSHW_LOGO_400mil
- H1, H2, H3, H4: footprint (none) -> Bus_Usb_Power:MountingHole_3mm
- J1: footprint (none) -> Bus_Usb_Power:Pin_Header_Straight_1x03
- N2: footprint (none) -> Bus_Usb_Power:Pin_Header_Straight_2x05_Shrouded
- N3, N4, N5, N6, N7: footprint (none) -> Bus_Usb_Power:5MM_TERMINAL_BLOCK_2_POS
- Q1, Q2: footprint (none) -> Bus_Usb_Power:TO-220_FET-GDS_Horizontal_LargePads
- R1: footprint (none) -> Bus_Usb_Power:Resistor_Horizontal_400
- R2, R3: footprint (none) -> Bus_Usb_Power:MF_R300
- SW1: footprint (none) -> Bus_Usb_Power:GF_426_0020
Changed lines of the file:
@@
 EESchema Schematic File Version 2
-LIBS:bus_power
+LIBS:bus_usb_power
 LIBS:power
 LIBS:device
@@
 LIBS:contrib
 LIBS:valves
-LIBS:bus_power-cache
+LIBS:bus_usb_power-cache
 EELAYER 25 0
 EELAYER END
@@
 F 0 "H1" H 4150 7250 50  0000 C CNN
 F 1 "3MM_HOLE" H 4200 6950 50  0000 C CNN
-F 2 "" H 4200 7100 60  0000 C CNN
+F 2 "Bus_Usb_Power:MountingHole_3mm" H 4200 7100 60  0001 C CNN
 F 3 "" H 4200 7100 60  0000 C CNN
 	1    4200 7100
@@
 F 0 "G1" H 6550 4350 60  0000 C CNN
 F 1 "OSHW_LOGO" H 6550 3975 60  0000 C CNN
-F 2 "" H 6550 4150 60  0000 C CNN
+F 2 "Bus_Usb_Power:OSHW_LOGO_400mil" H 6550 4150 60  0001 C CNN
 F 3 "" H 6550 4150 60  0000 C CNN
 	1    6550 4150
@@
 F 0 "N4" H 2500 2200 50  0000 C CNN
 F 1 "OSTTC020162" H 2500 1900 50  0000 C CNN
-F 2 "" H 2500 2050 60  0000 C CNN
+F 2 "Bus_Usb_Power:5MM_TERMINAL_BLOCK_2_POS" H 2500 2050 60  0001 C CNN
 F 3 "" H 2500 2050 60  0000 C CNN
 	1    2500 2050
@@
 F 0 "Q1" H 3975 1900 50  0000 C CNN
 F 1 "FQP47P06" H 3900 2275 50  0000 C CNN
-F 2 "" H 3900 2100 60  0000 C CNN
+F 2 "Bus_Usb_Power:TO-220_FET-GDS_Horizontal_LargePads" H 3900 2100 60  0001 C CNN
 F 3 "" H 3900 2100 60  0000 C CNN
 	1    3900 2100
@@
 F 0 "N5" H 2500 2600 50  0000 C CNN
 F 1 "OSTTC020162" H 2500 2300 50  0000 C CNN
-F 2 "" H 2500 2450 60  0000 C CNN
+F 2 "Bus_Usb_Power:5MM_TERMINAL_BLOCK_2_POS" H 2500 2450 60  0001 C CNN
 F 3 "" H 2500 2450 60  0000 C CNN
 	1    2500 2450
@@
 F 0 "R2" H 5000 2200 50  0000 C CNN
 F 1 "MF-R300" H 5000 1950 50  0000 C CNN
-F 2 "" H 5000 2100 60  0000 C CNN
+F 2 "Bus_Usb_Power:MF_R300" H 5000 2100 60  0001 C CNN
 F 3 "" H 5000 2100 60  0000 C CNN
 	1    5000 2100
@@
 F 0 "SW1" H 4500 5700 50  0000 C CNN
 F 1 "F-426-0020" H 4500 4950 50  0000 C CNN
-F 2 "" H 4500 5445 60  0000 C CNN
+F 2 "Bus_Usb_Power:GF_426_0020" H 4500 5445 60  0001 C CNN
 F 3 "" H 4500 5445 60  0000 C CNN
 	1    4500 5325
@@
 F 0 "N6" H 2500 6800 50  0000 C CNN
 F 1 "OSTTC020162" H 2500 6500 50  0000 C CNN
-F 2 "" H 2500 6650 60  0000 C CNN
+F 2 "Bus_Usb_Power:5MM_TERMINAL_BLOCK_2_POS" H 2500 6650 60  0001 C CNN
 F 3 "" H 2500 6650 60  0000 C CNN
 	1    2500 6650
@@
 F 0 "N7" H 2500 7200 50  0000 C CNN
 F 1 "OSTTC020162" H 2500 6900 50  0000 C CNN
-F 2 "" H 2500 7050 60  0000 C CNN
+F 2 "Bus_Usb_Power:5MM_TERMINAL_BLOCK_2_POS" H 2500 7050 60  0001 C CNN
 F 3 "" H 2500 7050 60  0000 C CNN
 	1    2500 7050
@@
 F 0 "Q2" H 3975 6400 50  0000 C CNN
 F 1 "FQP47P06" H 3900 6775 50  0000 C CNN
-F 2 "" H 3900 6600 60  0000 C CNN
+F 2 "Bus_Usb_Power:TO-220_FET-GDS_Horizontal_LargePads" H 3900 6600 60  0001 C CNN
 F 3 "" H 3900 6600 60  0000 C CNN
 	1    3900 6600
@@
 F 0 "N3" H 2500 1800 50  0000 C CNN
 F 1 "OSTTC020162" H 2500 1500 50  0000 C CNN
-F 2 "" H 2500 1650 60  0000 C CNN
+F 2 "Bus_Usb_Power:5MM_TERMINAL_BLOCK_2_POS" H 2500 1650 60  0001 C CNN
 F 3 "" H 2500 1650 60  0000 C CNN
 	1    2500 1650
@@
 F 0 "R3" H 5000 6700 50  0000 C CNN
 F 1 "MF-R300" H 5000 6450 50  0000 C CNN
-F 2 "" H 5000 6600 60  0000 C CNN
+F 2 "Bus_Usb_Power:MF_R300" H 5000 6600 60  0001 C CNN
 F 3 "" H 5000 6600 60  0000 C CNN
 	1    5000 6600
@@
 F 0 "J1" H 1950 4550 50  0000 C CNN
 F 1 "TERMINATE_JUMPER" H 2000 4150 50  0000 C CNN
-F 2 "" H 2000 4350 60  0000 C CNN
+F 2 "Bus_Usb_Power:Pin_Header_Straight_1x03" H 2000 4350 60  0001 C CNN
 F 3 "" H 2000 4350 60  0000 C CNN
 	1    2000 4350
@@
 F 0 "R1" H 2600 4450 50  0000 C CNN
 F 1 "120 1%" H 2600 4250 50  0000 C CNN
-F 2 "" H 2625 4350 60  0000 C CNN
+F 2 "Bus_Usb_Power:Resistor_Horizontal_400" H 2625 4350 60  0001 C CNN
 F 3 "" H 2625 4350 60  0000 C CNN
 	1    2600 4350
@@
 F 0 "H2" H 4150 7700 50  0000 C CNN
 F 1 "3MM_HOLE" H 4200 7400 50  0000 C CNN
-F 2 "" H 4200 7550 60  0000 C CNN
+F 2 "Bus_Usb_Power:MountingHole_3mm" H 4200 7550 60  0001 C CNN
 F 3 "" H 4200 7550 60  0000 C CNN
 	1    4200 7550
@@
 F 0 "H3" H 4600 7500 50  0000 C CNN
 F 1 "3MM_HOLE" H 4650 7200 50  0000 C CNN
-F 2 "" H 4650 7350 60  0000 C CNN
+F 2 "Bus_Usb_Power:MountingHole_3mm" H 4650 7350 60  0001 C CNN
 F 3 "" H 4650 7350 60  0000 C CNN
 	1    4650 7350
@@
 F 0 "H4" H 4600 7950 50  0000 C CNN
 F 1 "3MM_HOLE" H 4650 7650 50  0000 C CNN
-F 2 "" H 4650 7800 60  0000 C CNN
+F 2 "Bus_Usb_Power:MountingHole_3mm" H 4650 7800 60  0001 C CNN
 F 3 "" H 4650 7800 60  0000 C CNN
 	1    4650 7800
@@
 F 0 "N2" H 2250 4700 50  0000 C CNN
 F 1 "BUS_MASTER_HEADER" H 2400 5800 50  0000 C CNN
-F 2 "" H 2400 5250 60  0000 C CNN
+F 2 "Bus_Usb_Power:Pin_Header_Straight_2x05_Shrouded" H 2400 5250 60  0001 C CNN
 F 3 "" H 2400 5250 60  0000 C CNN
 	1    2400 5250

Commit message: Initial layout of Rev. A is complete.
Parts:
- added N1, N8: AY-Y1008-2-R, Bus_Usb_Power:DUAL_USB_A, symbol DUAL_USB_A
- added R4, R5, R6, R7: 200, Bus_Usb_Power:Resistor_Horizontal_400, symbol R_HORIZ
- added VR1: D24V25F6, Bus_Usb_Power:D24V25F6, symbol D24V25F6
- added VR2: OKI-78SR-5/1.5-W36-C, symbol VOLTAGE_REGULATOR_123
- added VR3: OKI-78SR-5/1.5-W36-C, ~, symbol VOLTAGE_REGULATOR_123
- N3, N4, N5, N6, N7: value OSTTC020162 -> 2POS_5MM_TERM_BLK
Connections:
- net labels added: LPWR5, USB1_5V, USB2_5V
- wire segments 57 -> 112
- no-connect marks 3 -> 8
Other:
- note added: "6A Polyfuse"
- note added: "DC-DC Converter 5V@1.5A"
- note added: "Dual Stacked USB A\nCharging Port"
- note added: "Note: When D24V25F6 is installed, install a jumper\nbetween pin 7 and pin 8 to short LGND and MGND\ntogether. When D24V25F6 is not installed, jumper\nbetween pin 9 and 10 to route LPWR3 connector to SW1."
- note added: "On_Board\nLogic Supply"
- note added: "Polarity Protection"
- note added: "Pololu DC-DC Converter 6V@2.5A"
- note added: "Power Switch"
- moved on the sheet: G1, J1, N2, R1, SW1

Commit message: Rev A. read for manufacture.
Parts:
- VR2: footprint (none) -> Bus_Usb_Power:OKI_DC_TO_DC_CONNECTOR
- VR3: footprint ~ -> Bus_Usb_Power:OKI_DC_TO_DC_CONNECTOR
Connections:
- net LGND: no longer H1.1 (GND), H2.1 (GND), H3.1 (GND), H4.1 (GND)
- no-connect marks 8 -> 12
Other:
- moved on the sheet: H1, H2, H3, H4
Changed lines of the file:
@@
 Sheet 1 1
 Title "Bus USB Power"
-Date "Fri 09 Jan 2015"
+Date "Tue 13 Jan 2015"
 Rev "A"
 Comp ""
@@
 L 3MM_HOLE H1
 U 1 1 53AA33AA
-P 4200 7100
-F 0 "H1" H 4150 7250 50  0000 C CNN
-F 1 "3MM_HOLE" H 4200 6950 50  0000 C CNN
-F 2 "Bus_Usb_Power:MountingHole_3mm" H 4200 7100 60  0001 C CNN
-F 3 "" H 4200 7100 60  0000 C CNN
-	1    4200 7100
+P 4500 7300
+F 0 "H1" H 4450 7450 50  0000 C CNN
+F 1 "3MM_HOLE" H 4500 7150 50  0000 C CNN
+F 2 "Bus_Usb_Power:MountingHole_3mm" H 4500 7300 60  0001 C CNN
+F 3 "" H 4500 7300 60  0000 C CNN
+	1    4500 7300
 	1    0    0    -1
 $EndComp
@@
 L 3MM_HOLE H2
 U 1 1 53E91440
-P 4200 7550
-F 0 "H2" H 4150 7700 50  0000 C CNN
-F 1 "3MM_HOLE" H 4200 7400 50  0000 C CNN
-F 2 "Bus_Usb_Power:MountingHole_3mm" H 4200 7550 60  0001 C CNN
-F 3 "" H 4200 7550 60  0000 C CNN
-	1    4200 7550
+P 4500 7700
+F 0 "H2" H 4450 7850 50  0000 C CNN
+F 1 "3MM_HOLE" H 4500 7550 50  0000 C CNN
+F 2 "Bus_Usb_Power:MountingHole_3mm" H 4500 7700 60  0001 C CNN
+F 3 "" H 4500 7700 60  0000 C CNN
+	1    4500 7700
 	1    0    0    -1
 $EndComp
@@
 L 3MM_HOLE H3
 U 1 1 53E914C5
-P 4650 7350
-F 0 "H3" H 4600 7500 50  0000 C CNN
-F 1 "3MM_HOLE" H 4650 7200 50  0000 C CNN
-F 2 "Bus_Usb_Power:MountingHole_3mm" H 4650 7350 60  0001 C CNN
-F 3 "" H 4650 7350 60  0000 C CNN
-	1    4650 7350
+P 5000 7300
+F 0 "H3" H 4950 7450 50  0000 C CNN
+F 1 "3MM_HOLE" H 5000 7150 50  0000 C CNN
+F 2 "Bus_Usb_Power:MountingHole_3mm" H 5000 7300 60  0001 C CNN
+F 3 "" H 5000 7300 60  0000 C CNN
+	1    5000 7300
 	1    0    0    -1
 $EndComp
@@
 L 3MM_HOLE H4
 U 1 1 53E91517
-P 4650 7800
-F 0 "H4" H 4600 7950 50  0000 C CNN
-F 1 "3MM_HOLE" H 4650 7650 50  0000 C CNN
-F 2 "Bus_Usb_Power:MountingHole_3mm" H 4650 7800 60  0001 C CNN
-F 3 "" H 4650 7800 60  0000 C CNN
-	1    4650 7800
+P 5000 7700
+F 0 "H4" H 4950 7850 50  0000 C CNN
+F 1 "3MM_HOLE" H 5000 7550 50  0000 C CNN
+F 2 "Bus_Usb_Power:MountingHole_3mm" H 5000 7700 60  0001 C CNN
+F 3 "" H 5000 7700 60  0000 C CNN
+	1    5000 7700
 	1    0    0    -1
 $EndComp
@@
 F 0 "VR2" H 7000 3600 50  0000 C CNN
 F 1 "OKI-78SR-5/1.5-W36-C" H 7500 3250 50  0000 C CNN
-F 2 "" H 7000 3400 60  0000 C CNN
+F 2 "Bus_Usb_Power:OKI_DC_TO_DC_CONNECTOR" H 7000 3400 60  0001 C CNN
 F 3 "" H 7000 3400 60  0000 C CNN
 	1    7000 3400
@@
 	5400 2100 6300 2100
 Wire Wire Line
-	2800 7100 4000 7100
-Wire Wire Line
-	3900 6950 3900 7800
-Wire Wire Line
 	2800 6600 3600 6600
 Wire Wire Line
@@
 	3300 4400 3300 2500
 Connection ~ 3300 2500
-Connection ~ 3900 7100
-Wire Wire Line
-	3900 7550 4000 7550
-Wire Wire Line
-	3900 7800 4450 7800
-Connection ~ 3900 7550
-Wire Wire Line
-	4450 7350 3900 7350
-Connection ~ 3900 7350
 Wire Wire Line
 	2900 6700 2900 7100
@@
 F 0 "VR3" H 7000 5200 50  0000 C CNN
 F 1 "OKI-78SR-5/1.5-W36-C" H 7500 4850 50  0000 C CNN
-F 2 "~" H 7000 5000 60  0000 C CNN
+F 2 "Bus_Usb_Power:OKI_DC_TO_DC_CONNECTOR" H 7000 5000 60  0000 C CNN
 F 3 "" H 7000 5000 60  0000 C CNN
 	1    7000 5000
@@
 Text Label 7600 4900 0    60   ~ 0
 USB2_5V
+NoConn ~ 4800 7300
+NoConn ~ 4800 7700
+NoConn ~ 4300 7300
+NoConn ~ 4300 7700
+Wire Wire Line
+	2800 7100 3900 7100
+Wire Wire Line
+	3900 7100 3900 6950
 $EndSCHEMATC
