File: rev_b/bus_usb_power.sch (KiCad schematic (older format))
At the start: 27 parts, among them J1 TERMINATE_JUMPER, Q1 FQP47P06, Q2 FQP47P06, SW1 F-426-0020

Commit message: Rev. B is looking pretty good.
Parts:
- removed N1: AY-Y1008-2-R, Bus_Usb_Power:DUAL_USB_A, symbol DUAL_USB_A
- removed N6, N7: 2POS_5MM_TERM_BLK, Bus_Usb_Power:5MM_TERMINAL_BLOCK_2_POS, symbol POWER_CONNECTOR
- removed R3: MF-R300, Bus_Usb_Power:MF_R300, symbol RESETABLE_FUSE
- removed R6, R7: 200, Bus_Usb_Power:Resistor_Horizontal_400, symbol R_HORIZ
- removed VR1: D24V25F6, Bus_Usb_Power:D24V25F6, symbol D24V25F6
- removed VR2, VR3: OKI-78SR-5/1.5-W36-C, Bus_Usb_Power:OKI_DC_TO_DC_CONNECTOR, symbol VOLTAGE_REGULATOR_123
- added J1: POWER_SELECT, Bus_Usb_Power:Pin_Header_Straight_1x03, symbol POWER_SELECT
- added N3: USB_B, Bus_Usb_Power:USB_B, symbol USB_B
- added TP1, TP2, TP3, TP4, TP5: TEST_POINT, Bus_Usb_Power:Pin_Header_Straight_1x01, symbol TEST_POINT
- added VR1: S18V20F5, Bus_Usb_Power:S18V20Fx, symbol V18V20Fx
- added VR2: S7VVF5, Bus_Usb_Power:Pin_Header_Straight_1x04, symbol S7VxFx
- added VR3: S18V20ALV, Bus_Usb_Power:S18V20Fx, symbol V18V20Fx
- added VR4, VR6: S7V8A, Bus_Usb_Power:Pin_Header_Straight_1x04, symbol S7VxFx
- added VR5: S18V20F6, Bus_Usb_Power:S18V20Fx, symbol V18V20Fx
- renumbered J1 to J2, N5 to N1, N4 to N2, N8 to N4, N3 to N5, N2 to N6, Q2 to Q1, Q1 to Q2, R2 to R1, R4 to R2, R5 to R3, R1 to R4
Connections:
- net labels added: BAT+, BAT-, BAT_SW, BPWR1, BPWR2, FUSE_IN, FUSE_OUT, GND, LPWR, PWRCOM, USB_5V, USB_5V_IN
- net labels removed: LGND, LPWR1, LPWR2, LPWR3, LPWR4, LPWR5, MGND, MPWR0, MPWR1, MPWR2, MPWR3, MPWR4, USB1_5V, USB2_5V
- wire segments 111 -> 127
- no-connect marks 12 -> 15
Other:
- note added: "3A Polyfuse"
- note added: "Battery Input"
- note added: "Bus Termination"
- note added: "Switched Battery"
- note added: "USB Power In"
- note removed: "6A Polyfuse"
- note removed: "DC-DC Converter 5V@1.5A"
- note removed: "Daisy Chain\nMotor Power"
- note removed: "Logic Power\nDaisy Chain"
- note removed: "Logic Power\nInput"
- note removed: "Motor Power\nInput"
- note removed: "Note: When D24V25F6 is installed, install a jumper\nbetween pin 5 and pin 7 to short LGND and MGND\ntogether. When D24V25F6 is not installed, jumper\nbetween pin 9 and 10 to route LPWR3 connector to SW1."
- note removed: "On_Board\nLogic Supply"
- note removed: "Pololu DC-DC Converter 6V@2.5A"
- note removed: "Power Switch"
- moved on the sheet: G1, J2, N1, N2, N4, N5, N6, Q1, Q2, R1, R2, R3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

Commit message: More fine tuning of Rev. B
Connections:
- net BPWR2: no longer N5.1 (-), N6.10 (BPWR2), N6.9 (BPWR1)
- new net BPWR3: N5.1 (-), N6.10 (BPWR2), N6.9 (BPWR1)
Changed lines of the file:
@@
 	9300 2500 9600 2500
 Text Label 9300 3900 0    50   ~ 0
-BPWR2
+BPWR3
 Text Notes 9300 5650 0    50   ~ 0
 Bus Termination
