File: rev_b/$bus_usb_power.sch (KiCad schematic (older format))
At the start: 27 parts, among them J1 TERMINATE_JUMPER, Q1 FQP47P06, Q2 FQP47P06, SW1 F-426-0020

Commit message: Mid-point to a fairly major change.
Parts:
- removed VR2, VR3: OKI-78SR-5/1.5-W36-C, Bus_Usb_Power:OKI_DC_TO_DC_CONNECTOR, symbol VOLTAGE_REGULATOR_123
Changed lines of the file:
@@
 MGND
-$Comp
-L VOLTAGE_REGULATOR_123 VR2
-U 1 1 54B03369
-P 7000 3400
-F 0 "VR2" H 7000 3600 50  0000 C CNN
-F 1 "OKI-78SR-5/1.5-W36-C" H 7500 3250 50  0000 C CNN
-F 2 "Bus_Usb_Power:OKI_DC_TO_DC_CONNECTOR" H 7000 3400 60  0001 C CNN
-F 3 "" H 7000 3400 60  0000 C CNN
-	1    7000 3400
-	1    0    0    -1
-$EndComp
 $Comp
 L DUAL_USB_A N8
@@
 Text Notes 4200 4200 0    50   ~ 0
 Power Switch
-$Comp
-L VOLTAGE_REGULATOR_123 VR3
-U 1 1 54B17410
-P 7000 5000
-F 0 "VR3" H 7000 5200 50  0000 C CNN
-F 1 "OKI-78SR-5/1.5-W36-C" H 7500 4850 50  0000 C CNN
-F 2 "Bus_Usb_Power:OKI_DC_TO_DC_CONNECTOR" H 7000 5000 60  0001 C CNN
-F 3 "" H 7000 5000 60  0000 C CNN
-	1    7000 5000
-	1    0    0    -1
-$EndComp
 Wire Wire Line
 	8200 5500 9100 5500
