File: rev_b/bus_usb_power.kicad_pcb (KiCad board)
At the start: 2 copper layers, 100 x 50 mm, 27 parts, among them J1 TERMINATE_JUMPER, Q1 FQP47P06, Q2 FQP47P06, SW1 F-426-0020

Commit message: Fixed a whole bunch of issues.
Parts:
- moved R6 10.2 mm to (157.5, 127.6), turned to 180 degrees
- moved R5 5.08 mm to (157.5, 117.5)
- moved R4 5.08 mm to (157.5, 122.6)
- turned N1 to 180 degrees
- turned N8 to 180 degrees
Connections:
- N1 pad 10: /MGND -> /LGND
- N1 pad 11: /MGND -> /LGND
- N1 pad 12: /MGND -> /LGND
- N1 pad 4: /MGND -> /LGND
- N1 pad 8: /MGND -> /LGND
- N1 pad 9: /MGND -> /LGND
- N8 pad 10: /MGND -> /LGND
- N8 pad 11: /MGND -> /LGND
- N8 pad 12: /MGND -> /LGND
- N8 pad 4: /MGND -> /LGND
- N8 pad 8: /MGND -> /LGND
- N8 pad 9: /MGND -> /LGND
- VR2 pad 1: /LPWR4 -> /LPWR5
- VR2 pad 2: /MGND -> /LGND
- VR3 pad 1: /LPWR4 -> /LPWR5
- VR3 pad 2: /MGND -> /LGND
Routing:
- net /LGND: track 142.0 -> 235.0 mm
- net /MGND: track 184.3 -> 114.8 mm
- net /LPWR4: track 55.4 -> 12.7 mm
- net Net-(N1-Pad3): track 65.4 -> 38.1 mm
- net Net-(N1-Pad2): track 71.0 -> 46.2 mm
- net Net-(N8-Pad7): track 28.5 -> 37.4 mm
- net Net-(N8-Pad2): track 22.3 -> 16.2 mm
- net Net-(N1-Pad7): track 46.2 -> 51.1 mm
- net /USB1_5V: track 13.4 -> 8.65 mm
- net /USB2_5V: track 13.4 -> 8.65 mm
- net Net-(N1-Pad6): track 37.0 -> 40.0 mm
- net Net-(N8-Pad6): track 21.9 -> 23.9 mm
- net /LPWR5: track 70.9 -> 72.5 mm
- net Net-(N8-Pad3): track 30.9 -> 29.9 mm
Other:
- board text added: "Bus USB Power Rev. B 20Jan2015 Copyright (c) 2015 by Wayne Gramlich"
- board text added: "Rev. B 20Jan2015"
- board text removed: "Bus USB Power Rev. A 13Jan2015 (c) Gramlich"
- board text removed: "Rev. A 13Jan2015"

Commit message: Mid-point to a fairly major change.
Other:
- board text added: "TERM"
- board text removed: "Term"
Changed lines of the file:
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@@
   (gr_line (start 200 100) (end 200 150) (angle 90) (layer F.SilkS) (width 0.2032))
   (gr_line (start 100 100) (end 200 100) (angle 90) (layer F.SilkS) (width 0.2032))
-  (gr_text Term (at 114.3 146.685) (layer F.SilkS)
+  (gr_text TERM (at 114.3 146.685) (layer F.SilkS)
     (effects (font (size 1.016 1.016) (thickness 0.2032)))
   )

Commit message: Rev. B is looking pretty good.
Parts:
- removed N7: 2POS_5MM_TERM_BLK, Bus_Usb_Power:5MM_TERMINAL_BLOCK_2_POS
- removed N8: AY-Y1008-2-R, Bus_Usb_Power:DUAL_USB_A
- removed R5, R6, R7: 200, Bus_Usb_Power:Resistor_Horizontal_400
- added J2: TERMINATE_JUMPER, Bus_Usb_Power:Pin_Header_Straight_1x03, F.Cu at (104.8, 137.2)
- added TP1: TEST_POINT, Bus_Usb_Power:Pin_Header_Straight_1x01, F.Cu at (103.5, 113.0)
- added TP2: TEST_POINT, Bus_Usb_Power:Pin_Header_Straight_1x01, F.Cu at (106.7, 113.0)
- added TP3: TEST_POINT, Bus_Usb_Power:Pin_Header_Straight_1x01, F.Cu at (196.8, 135.3)
- added TP4: TEST_POINT, Bus_Usb_Power:Pin_Header_Straight_1x01, F.Cu at (146.1, 146.1)
- added TP5: TEST_POINT, Bus_Usb_Power:Pin_Header_Straight_1x01, F.Cu at (135.3, 148.6)
- added VR4: S7V8A, Bus_Usb_Power:Pin_Header_Straight_1x04, F.Cu at (142.2, 134.6)
- added VR5: S18V20F6, Bus_Usb_Power:S18V20Fx, F.Cu at (120.7, 121.9)
- added VR6: S7V8A, Bus_Usb_Power:Pin_Header_Straight_1x04, F.Cu at (120.7, 134.6)
- J1: value TERMINATE_JUMPER -> POWER_SELECT
- N1: value AY-Y1008-2-R -> 2POS_5MM_TERM_BLK; footprint Bus_Usb_Power:DUAL_USB_A -> Bus_Usb_Power:5MM_TERMINAL_BLOCK_2_POS
- N2: value BUS_MASTER_HEADER -> 2POS_5MM_TERM_BLK; footprint Bus_Usb_Power:Pin_Header_Straight_2x05_Shrouded -> Bus_Usb_Power:5MM_TERMINAL_BLOCK_2_POS
- N3: value 2POS_5MM_TERM_BLK -> USB_B; footprint Bus_Usb_Power:5MM_TERMINAL_BLOCK_2_POS -> Bus_Usb_Power:USB_B
- N4: value 2POS_5MM_TERM_BLK -> AY-Y1008-2-R; footprint Bus_Usb_Power:5MM_TERMINAL_BLOCK_2_POS -> Bus_Usb_Power:DUAL_USB_A
- N6: value 2POS_5MM_TERM_BLK -> BUS_MASTER_HEADER; footprint Bus_Usb_Power:5MM_TERMINAL_BLOCK_2_POS -> Bus_Usb_Power:Pin_Header_Straight_2x05_Shrouded
- R1: value 120 1% -> MF-R300; footprint Bus_Usb_Power:Resistor_Horizontal_400 -> Bus_Usb_Power:MF_R300
- R2, R3: value MF-R300 -> 200; footprint Bus_Usb_Power:MF_R300 -> Bus_Usb_Power:Resistor_Horizontal_400
- R4: value 200 -> 120 1%
- VR1: value D24V25F6 -> S18V20F5; footprint Bus_Usb_Power:D24V25F6 -> Bus_Usb_Power:S18V20Fx
- VR2: value OKI-78SR-5/1.5-W36-C -> S7VVF5; footprint Bus_Usb_Power:OKI_DC_TO_DC_CONNECTOR -> Bus_Usb_Power:Pin_Header_Straight_1x04
- VR3: value OKI-78SR-5/1.5-W36-C -> S18V20ALV; footprint Bus_Usb_Power:OKI_DC_TO_DC_CONNECTOR -> Bus_Usb_Power:S18V20Fx
- moved N6 91.7 mm to (104.8, 125.1), turned to 270 degrees
- moved N2 64.9 mm to (166.4, 148.0), turned to 0 degrees
- moved N5 51.8 mm to (128.3, 148.0), turned to 0 degrees
- moved R3 49.1 mm to (141.7, 109.7), turned to 0 degrees
- moved R4 46.3 mm to (112.0, 131.0), turned to 270 degrees
- moved R1 42.8 mm to (154.3, 146.1), turned to 180 degrees
- moved VR1 40.0 mm to (163.8, 121.9), turned to 90 degrees
- moved SW1 38.9 mm to (187.3, 125.7)
- moved N3 36.2 mm to (181.6, 139.7), turned to 0 degrees
- moved N1 34.7 mm to (114.9, 148.0), turned to 0 degrees
- moved R2 30.5 mm to (141.7, 129.0), turned to 0 degrees
- moved VR2 28.7 mm to (163.6, 134.6)
- moved Q2 27.0 mm to (170.8, 113.0)
- moved J1 25.8 mm to (139.7, 146.1), turned to 180 degrees
- moved VR3 22.2 mm to (142.2, 121.9), turned to 90 degrees
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Connections:
- net /MPWR1 renamed /USB_5V_IN
- J1 pad 1: Net-(J1-Pad1) -> /FUSE_IN
- J1 pad 2: Net-(J1-Pad2) -> /BPWR2
- J1 pad 3: (no net) -> /BPWR1
- N1 pad 1: /USB2_5V -> /GND
- N1 pad 2: Net-(N1-Pad2) -> /BAT_SW
- N2 pad 1: /LPWR5 -> /BAT-
- N2 pad 2: /LPWR5 -> /BAT+
- N3 pad 2: /MPWR0 -> (no net)
- N4 pad 1: /MGND -> /USB_5V
- N4 pad 2: /MPWR0 -> Net-(N4-Pad2)
- N5 pad 1: /MGND -> /BPWR2
- N5 pad 2: /MPWR0 -> /BPWR2
- N6 pad 1: /LGND -> /LPWR
- N6 pad 2: /LPWR1 -> /LPWR
- Q1 pad G: /MGND -> /GND
- Q1 pad S: /MPWR2 -> /PWRCOM
- Q2 pad D: /LPWR1 -> /BAT_SW
- Q2 pad G: /LGND -> /GND
- Q2 pad S: /LPWR2 -> /PWRCOM
- R1 pad 1: Net-(J1-Pad2) -> /PWRCOM
- R1 pad 2: Net-(N2-Pad6) -> /FUSE_IN
- R2 pad 1: /MPWR2 -> Net-(N4-Pad2)
- R2 pad 2: /MPWR3 -> Net-(N4-Pad3)
- R3 pad 1: /LPWR2 -> Net-(N4-Pad6)
- R3 pad 2: /LPWR3 -> Net-(N4-Pad7)
- R4 pad 1: Net-(N8-Pad2) -> Net-(N6-Pad6)
- SW1 pad 1: /MPWR3 -> /BAT_SW
- SW1 pad 2: /MPWR4 -> /BAT+
- SW1 pad 4: /LPWR4 -> /GND
- SW1 pad 5: /LPWR5 -> /BAT-
- VR1 pad 1: (no net) -> /GND
- VR1 pad 10: /LPWR4 -> (no net)
- VR1 pad 2: (no net) -> /GND
- VR1 pad 3: (no net) -> /FUSE_IN
- VR1 pad 4: /MPWR3 -> /FUSE_IN
- VR1 pad 5: /MGND -> (no net)
- VR1 pad 6: /MGND -> /GND
- VR1 pad 7: /LGND -> /GND
- VR1 pad 8: /MGND -> /USB_5V
- VR1 pad 9: /LPWR3 -> /USB_5V
- VR2 pad 1: /LPWR5 -> /USB_5V
- VR2 pad 2: /LGND -> /GND
- VR2 pad 3: /USB1_5V -> /FUSE_IN
- VR3 pad 1: /LPWR5 -> /GND
- VR3 pad 2: /LGND -> /GND
- VR3 pad 3: /USB2_5V -> /FUSE_IN
Routing:
- net /LGND: track 235.0 -> 0.00 mm
- net /USB_5V: track 0.00 -> 133.5 mm
- net /MGND: track 114.8 -> 0.00 mm
- net /BAT_SW: track 0.00 -> 104.5 mm
- net /FUSE_IN: track 0.00 -> 75.1 mm
- net /LPWR5: track 72.5 -> 0.00 mm, vias 1 -> 0
- net Net-(N4-Pad2): track 0.00 -> 63.0 mm
- net /LPWR: track 0.00 -> 56.6 mm
- net Net-(N4-Pad6): track 0.00 -> 56.1 mm
- net /PWRCOM: track 0.00 -> 52.4 mm
- net /MPWR4: track 51.5 -> 0.00 mm
- net /MPWR3: track 51.2 -> 0.00 mm
- net Net-(N1-Pad7): track 51.1 -> 0.00 mm
- net /BPWR2: track 0.00 -> 50.4 mm
- net /BPWR1: track 0.00 -> 47.7 mm
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- added copper zone on B.Cu, net /GND
- added copper zone on F.Cu, net /GND
Other:
- board text added: "BAT"
- board text added: "BUS_USB_POWER"
- board text added: "ESTOP"
- board text added: "POWER ON/OFF"
- board text added: "REV. B (C) 2015 GRAMLICH"
- board text added: "SW-BAT"
- board text added: "TERMINATE"
- board text removed: "1"
- board text removed: "Bus USB Power Rev. B 20Jan2015 Copyright (c) 2015 by Wayne Gramlich"
- board text removed: "Bus_USB_Power"
- board text removed: "CHAIN"
- board text removed: "E-STOP"
- board text removed: "IN"
- board text removed: "INPUT"
- board text removed: "LPWR"
- board text removed: "MPWR"
- board text removed: "Rev. B 20Jan2015"
- board text removed: "TERM"

Commit message: More fine tuning of Rev. B
Parts:
- moved J1 1.27 mm to (141.0, 146.1)
- moved TP3 0.90 mm to (197.5, 134.6)
- moved TP2 0.64 mm to (106.0, 113.0)
- moved TP1 0.63 mm to (102.9, 113.0)
- moved TP4 0.63 mm to (146.7, 146.1)
Connections:
- N5 pad 1: /BPWR2 -> /BPWR3
- N6 pad 10: /BPWR2 -> /BPWR3
- N6 pad 9: /BPWR2 -> /BPWR3
Routing:
- net /BPWR2: track 50.4 -> 12.3 mm
- net /BPWR3: track 0.00 -> 35.1 mm
- net Net-(N4-Pad2): track 63.0 -> 59.2 mm
- net Net-(N4-Pad6): track 56.1 -> 54.9 mm
- net /FUSE_IN: track 75.1 -> 74.2 mm
- net /LPWR: track 56.6 -> 57.5 mm
- net /USB_5V: track 133.5 -> 134.2 mm
- net Net-(N4-Pad3): track 47.4 -> 46.8 mm
- net /BPWR1: track 47.7 -> 48.2 mm
Other:
- board text added: "BPWR REGULATOR"
- board text added: "Bus USB Power Rev. B 24Jan2014 Copyright (c) 2015 by Wayne Gramlich"
- board text added: "LPWR REGULATOR"
- board text added: "REG/BAT"
- board text added: "REV. B 24JAN2015 (C) 2015"
- board text added: "USB PWR 1-2 AMPS"
- board text added: "USB PWR IN"
- board text added: "USB REGULATOR"
- board text removed: "REV. B (C) 2015 GRAMLICH"
